File: hardware/rev_a/squall-blees-board.sch (EAGLE design)
At the start: 7 parts, among them J1 SQUALL_HEADER, J4 HIROSE-DF40C-10DP-0.4V, J5 HIROSE-DF40C-10DP-0.4V

Commit message: Work on circuit board
Parts:
- removed J2, J3: (no value), pinhead:PINHD-2X8
- removed J6: (no value), pinhead:PINHD-1X1
- added C1: 10uF, passives:CAPACITOR0603_CAP
- added C2, C3, C4: 100nF, passives:CAPACITOR
- added U$1: TSL2560DFN, blees:TSL2560DFN
- added U1: HTU21DDFN, blees:HTU21DDFN
- added U2: LPS331APQFN, blees:LPS331APQFN
Connections:
- net 5V: no longer J6.1
- net A5: no longer J3.5, J3.6
- net A6: no longer J3.3, J3.4
- net A7: no longer J3.1, J3.2
- net GND: now also C1.2, C2.2, C3.2, C4.2, U$1.ADDR_SEL, U$1.GND, U1.GND, U1.PAD, U2.GND@12, U2.GND@13, U2.GND@16, U2.GND@5, U2.RSV, U2.SA0; no longer J2.15, J2.16
- net MISO: no longer J3.10, J3.9
- net MOSI: no longer J3.7, J3.8
- net P22: no longer J2.3, J2.4
- net P23: no longer J2.5, J2.6
- net P24: no longer J2.7, J2.8
- net P25: no longer J2.10, J2.9
- net SCL: now also U$1.SCL, U1.SCK, U2.SCL; no longer J2.13, J2.14
- net SCLK: no longer J3.11, J3.12
- net SDA: now also U$1.SDA, U1.SDA, U2.SDA; no longer J2.11, J2.12
- net SWDCLK: no longer J3.13, J3.14
- net SWDIO/!RESET: no longer J3.15, J3.16
- net VCC: now also C1.1, C2.1, C3.1, C4.1, U$1.VDD, U1.VDD, U2.CS, U2.VCCA, U2.VDD, U2.VDD_IO; no longer J2.1, J2.2
Other:
- note removed: "5V"
- note removed: "Left"
- note removed: "Right"

Commit message: Board finished
Parts:
- removed LOGO1: UMICH_SOLID_TINY, logos:UMICH_SOLID_TINY
- removed U1: HTU21DDFN, blees:HTU21DDFN
- added R1, R2: 2kΩ, passives:RESISTOR0402_RES
- added TEMP/HUMID: HTU21DDFN, blees:HTU21DDFN
- renumbered U$1 to LIGHT, U2 to PRESSURE
Connections:
- net GND: now also TEMP/HUMID.GND, TEMP/HUMID.PAD; no longer U1.GND, U1.PAD
- net SCL: now also R2.1, TEMP/HUMID.SCK; no longer U1.SCK
- net SDA: now also R1.1, TEMP/HUMID.SDA; no longer U1.SDA
- net VCC: now also R1.2, R2.2, TEMP/HUMID.VDD; no longer U1.VDD
Other:
- moved on the sheet: C3
