File: hardware/rev_d/squall-blees-board.brd (EAGLE design)
At the start: 27.7 x 23.4 mm, 19 parts, among them J1 SQUALL_HEADER, J2 HIROSE-DF40C-10DP-0.4V, J3 HIROSE-DF40C-10DP-0.4V, J5 TC2030-JLINK-NL, U1 LPS331APQFN, U2 TSL2560DFN, U3 SI7021, U4 ADXL362

Commit message: BLEES PCB rev D. Panelized and packaged
Routing:
- net GND: vias 20 -> 21
Changed lines of the file:
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@@
 <via x="29.5656" y="13.4366" extent="1-16" drill="0.4064"/>
 <via x="28.2702" y="7.4676" extent="1-16" drill="0.4064"/>
+<via x="15.9258" y="12.6746" extent="1-16" drill="0.4064"/>
 </signal>
 <signal name="A6">
