File: hardware/blink/rev_a/blink.sch (EAGLE design)
At the start: 7 parts, among them J1 SQUALL_HEADER, J2 HIROSE-DF40C-10DP-0.4V, J3 HIROSE-DF40C-10DP-0.4V, J5 TC2030-JLINK-NL, U1 AMN41121

Commit message: updated PIR sensor part number
Parts:
- U1: DIGIKEY (none) -> 255-3065-ND
Changed lines of the file:
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@@
 <?xml version="1.0" encoding="utf-8"?>
 <!DOCTYPE eagle SYSTEM "eagle.dtd">
-<eagle version="6.5.0">
+<eagle version="6.6.0">
 <drawing>
 <settings>
@@
 <part name="R1" library="passives" deviceset="RESISTOR" device="0402_RES" value="1kΩ"/>
 <part name="P+9" library="supply1" deviceset="VCC" device=""/>
-<part name="U1" library="chips" deviceset="AMN" device="41121"/>
+<part name="U1" library="chips" deviceset="AMN" device="41121">
+<attribute name="DIGIKEY" value="255-3065-ND"/>
+</part>
 <part name="P+6" library="supply1" deviceset="VCC" device=""/>
 <part name="GND7" library="umich" deviceset="GND" device=""/>
